Commit message: Add wheels

File: description/core.xacro (robot description, xacro)
@@ -31,3 +31,31 @@
         </visual>
     </link>
+    <joint name="left_wheel_joint" type="continuous">
+        <parent link="base_link"/>
+        <child link="left_wheel"/>
+        <origin xyz="0 0.175 0" rpy="-${pi/2} 0 0"/>
+        <axis xyz="0 0 1"/>
+    </joint>
+    <link name="left_wheel">
+        <visual>
+            <geometry>
+                <cylinder radius="0.05" length="0.04"/>
+            </geometry>
+            <material name="black"/>
+        </visual>
+    </link>
+    <joint name="right_wheel_joint" type="continuous">
+        <parent link="base_link"/>
+        <child link="right_wheel"/>
+        <origin xyz="0 -0.175 0" rpy="${pi/2} 0 0"/>
+        <axis xyz="0 0 -1"/>
+    </joint>
+    <link name="right_wheel">
+        <visual>
+            <geometry>
+                <cylinder radius="0.05" length="0.04"/>
+            </geometry>
+            <material name="black"/>
+        </visual>
+    </link>
 </robot>

Commit message: Add caster wheel to robot

File: description/core.xacro (robot description, xacro)
@@ -59,3 +59,16 @@
         </visual>
     </link>
+    <joint name="caster_wheel_joint" type="fixed">
+        <parent link="chassis"/>
+        <child link="caster_wheel"/>
+        <origin xyz="0.24 0 0"/>
+    </joint>
+    <link name="caster_wheel">
+        <visual>
+            <geometry>
+                <sphere radius="0.05"/>
+            </geometry>
+            <material name="black"/>
+        </visual>
+    </link>
 </robot>

Commit message: Add collision to each links

File: description/core.xacro (robot description, xacro)
@@ -28,6 +28,12 @@
                 <box size="0.3 0.3 0.15"/>
             </geometry>
-            <material name="white"/>
+            <material name="orange"/>
         </visual>
+        <collision>
+            <origin xyz="0.15 0 0.075"/>
+            <geometry>
+                <box size="0.3 0.3 0.15"/>
+            </geometry>
+        </collision>
     </link>
     <joint name="left_wheel_joint" type="continuous">
@@ -44,4 +50,9 @@
             <material name="black"/>
         </visual>
+        <collision>
+            <geometry>
+                <cylinder radius="0.05" length="0.04"/>
+            </geometry>
+        </collision>
     </link>
     <joint name="right_wheel_joint" type="continuous">
@@ -58,4 +69,9 @@
             <material name="black"/>
         </visual>
+        <collision>
+            <geometry>
+                <cylinder radius="0.05" length="0.04"/>
+            </geometry>
+        </collision>
     </link>
     <joint name="caster_wheel_joint" type="fixed">
@@ -71,4 +87,9 @@
             <material name="black"/>
         </visual>
+        <collision>
+            <geometry>
+                <sphere radius="0.05"/>
+            </geometry>
+        </collision>
     </link>
 </robot>

Commit message: Add inertial to each links

File: description/core.xacro (robot description, xacro)
@@ -1,4 +1,5 @@
 <?xml version="1.0"?>
 <robot xmlns:xacro="http://www.ros.org/wiki/xacro">
+    <xacro:include filename="inertial_macros.xacro"/>
     <material name="white">
         <color rgba="1 1 1 1"/>
@@ -16,4 +17,5 @@
     <link name="base_link">
     </link>
+    <!-- Chassis -->
     <!-- origin is in the back, behind the 2 wheels -->
     <joint name="chassis_joint" type="fixed">
@@ -36,5 +38,9 @@
             </geometry>
         </collision>
+        <xacro:inertial_box mass="0.5" x="0.3" y="0.3" z="0.15">
+            <origin xyz="0.15 0 0.075" rpy="0 0 0"/>
+        </xacro:inertial_box>
     </link>
+    <!-- Left wheel -->
     <joint name="left_wheel_joint" type="continuous">
         <parent link="base_link"/>
@@ -55,5 +61,9 @@
             </geometry>
         </collision>
+        <xacro:inertial_cylinder mass="0.1" length="0.04" radius="0.05">
+            <origin xyz="0 0 0" rpy="0 0 0"/>
+        </xacro:inertial_cylinder>
     </link>
+    <!-- Right wheel -->
     <joint name="right_wheel_joint" type="continuous">
         <parent link="base_link"/>
@@ -74,5 +84,9 @@
             </geometry>
         </collision>
+        <xacro:inertial_cylinder mass="0.1" length="0.04" radius="0.05">
+            <origin xyz="0 0 0" rpy="0 0 0"/>
+        </xacro:inertial_cylinder>
     </link>
+    <!-- Caster wheel -->
     <joint name="caster_wheel_joint" type="fixed">
         <parent link="chassis"/>
@@ -92,4 +106,7 @@
             </geometry>
         </collision>
+        <xacro:inertial_sphere mass="0.1" radius="0.05">
+            <origin xyz="0 0 0" rpy="0 0 0"/>
+        </xacro:inertial_sphere>
     </link>
 </robot>

Commit message: Add drive control and obstacles

File: description/core.xacro (robot description, xacro)
@@ -44,4 +44,7 @@
         </xacro:inertial_box>
     </link>
+    <gazebo reference="chassis">
+        <material>Gazebo/Orange</material>
+    </gazebo>
     <!-- Left wheel -->
     <joint name="left_wheel_joint" type="continuous">
@@ -69,4 +72,7 @@
         </xacro:inertial_cylinder>
     </link>
+    <gazebo reference="left_wheel">
+        <material>Gazebo/Black</material>
+    </gazebo>
     <!-- Right wheel -->
     <joint name="right_wheel_joint" type="continuous">
@@ -94,4 +100,7 @@
         </xacro:inertial_cylinder>
     </link>
+    <gazebo reference="right_wheel">
+        <material>Gazebo/Black</material>
+    </gazebo>
     <!-- Caster wheel -->
     <joint name="caster_wheel_joint" type="fixed">
@@ -116,3 +125,9 @@
         </xacro:inertial_sphere>
     </link>
+    <gazebo reference="caster_wheel">
+        <!-- friction coefficience (near 0, almost frictionless) -->
+        <mu1 value="0.001"/>
+        <mu2 value="0.001"/>
+        <material>Gazebo/Black</material>
+    </gazebo>
 </robot>

File: description/robot.urdf.xacro (robot description, xacro)
@@ -2,3 +2,4 @@
 <robot xmlns:xacro="http://www.ros.org/wiki/xacro"  name="robot">
     <xacro:include filename="core.xacro"/>
+    <xacro:include filename="gz_controls.xacro"/>
 </robot>

Commit message: Add lidar simulation

File: description/core.xacro (robot description, xacro)
@@ -14,4 +14,7 @@
     <material name="black">
         <color rgba="0 0 0 1"/>
+    </material>
+    <material name="red">
+        <color rgba="1 0 0 1"/>
     </material>
     <!-- sits on the center of the 2 wheels as that is the center of rotation -->

File: description/gz_controls.xacro (robot description, xacro)
@@ -1,4 +1,4 @@
 <?xml version="1.0"?>
-<robot xmlns:xacro="http://www.ros.org/wiki/xacro"  name="robot">
+<robot xmlns:xacro="http://www.ros.org/wiki/xacro">
     <gazebo>
         <plugin name="diff_drive" filename="libgazebo_ros_diff_drive.so">

File: description/robot.urdf.xacro (robot description, xacro)
@@ -3,3 +3,4 @@
     <xacro:include filename="core.xacro"/>
     <xacro:include filename="gz_controls.xacro"/>
+    <xacro:include filename="lidar.xacro"/>
 </robot>

Commit message: Add ros2 nav

File: description/core.xacro (robot description, xacro)
@@ -21,4 +21,12 @@
     <link name="base_link">
     </link>
+    <!-- Base footprint -->
+     <joint name="base_footprint_link" type="fixed">
+        <parent link="base_link"/>
+        <child link="base_footprint"/>
+        <origin xyz="0 0 0" rpy="0 0 0"/>
+     </joint>
+     <link name="base_footprint">
+     </link>
     <!-- Chassis -->
     <!-- origin is in the back, behind the 2 wheels (hence -0.1 in the x axis) -->
